File: Modules/Modules.kicad_sch (KiCad schematic)
At the start: 41 parts, among them IC1 TMP126NDCKR, T1 2450FB15L0001E, U1 TPS62202DBV, U2 ESP32-WROOM-32D, U3 TPS62203DBV, U4 AT86RF233-ZU, U5 MCP3204, Y1 16M, Y2 40M

Commit message: First concept of the routed board
Parts:
- C1, C15, C20, C7: footprint Capacitor_THT:C_Radial_D8.0mm_H11.5mm_P3.50mm -> Capacitor_SMD:C_0402_1005Metric
- C2, C3, C4, C5, C6: footprint Capacitor_THT:C_Disc_D7.5mm_W2.5mm_P5.00mm -> Capacitor_SMD:C_0402_1005Metric
- R1, R2, R4, R6, R8: footprint Resistor_THT:R_Axial_DIN0207_L6.3mm_D2.5mm_P7.62mm_Horizontal -> Resistor_SMD:R_1210_3225Metric
- Y1, Y2: footprint Crystal:Crystal_HC52-6mm_Vertical -> Crystal:Crystal_SMD_0603-2Pin_6.0x3.5mm
Connections:
- net GNDA is gone; now on net GND: IC1.2 (GND), R3.2, R5.2, R7.2, U5.12 (AGND)
- net at U2.10 (IO25): now also U2.11 (IO26), U2.12 (IO27)
- net at U2.17 (SHD/SD2): now also U2.18 (SWP/SD3), U2.19 (SCS/CMD), U2.20 (SCK/CLK), U2.21 (SDO/SD0), U2.22 (SDI/SD1)
- net at U2.24 (IO2): now also U2.25 (IO0), U2.34 (RXD0/IO3), U2.35 (TXD0/IO1)
- net at U2.4 (SENSOR_VP): now also U2.5 (SENSOR_VN)
- net at U2.6 (IO34): now also U2.7 (IO35)
- net at U4.17 (CLKM): now also U4.24 (IRQ)
